Commit message: indy7 gazebo teleoperation

File: docker/docker_containers/indy7_container/share/catkin_ws/src/indy-ros/indy7_description/urdf/indy7.xacro (robot description, xacro)
@@ -4,5 +4,5 @@
 	<xacro:include filename="$(find indy7_description)/urdf/indy7.gazebo"/>
 	<xacro:property name="PI" value="3.1415926535897931"/>
-	<xacro:property name="indy_material" value="metal_grey"/>
+	<xacro:property name="indy_material" value="white"/>
 	<!-- <material name="grey"> <color rgba="0.5 0.5 0.5 1"/> </material> -->
 	<link name="link0">
@@ -194,5 +194,6 @@
 		<origin xyz="0 0 0.0775" rpy="0 0 0"/>
 		<axis xyz="0 0 1"/>
-		<limit effort="10" velocity="1" lower="-${175*PI/180}" upper="${175*PI/180}"/>
+		<limit effort="300" velocity="5" lower="-${175*PI/180}" upper="${175*PI/180}"/>
+		<dynamics damping="0.0" friction="0.0"/>
 	</joint>
 	<joint name="joint1" type="revolute">
@@ -201,5 +202,6 @@
 		<origin xyz="0 -0.10900000 0.22200000" rpy="${PI/2} ${PI/2} 0"/>
 		<axis xyz="0 0 1"/>
-		<limit effort="10" velocity="1" lower="-${175*PI/180}" upper="${175*PI/180}"/>
+		<limit effort="100" velocity="3" lower="-${175*PI/180}" upper="${175*PI/180}"/>
+		<dynamics damping="0.0" friction="0.0"/>
 	</joint>
 	<joint name="joint2" type="revolute">
@@ -208,5 +210,6 @@
 		<origin xyz="-0.45000000 +0.00000000 -0.03050000" rpy="0 0 0"/>
 		<axis xyz="0 0 1"/>
-		<limit effort="10" velocity="1" lower="-${175*PI/180}" upper="${175*PI/180}"/>
+		<limit effort="100" velocity="3" lower="-${175*PI/180}" upper="${175*PI/180}"/>
+		<dynamics damping="0.0" friction="0.0"/>
 	</joint>
 	<joint name="joint3" type="revolute">
@@ -215,5 +218,6 @@
 		<origin xyz="-0.26700000 +0.00000000 -0.07500000" rpy="-${PI/2} 0 ${PI/2}"/>
 		<axis xyz="0 0 1"/>
-		<limit effort="10" velocity="1" lower="-${175*PI/180}" upper="${175*PI/180}"/>
+		<limit effort="100" velocity="3" lower="-${175*PI/180}" upper="${175*PI/180}"/>
+		<dynamics damping="0.0" friction="0.0"/>
 	</joint>
 	<joint name="joint4" type="revolute">
@@ -222,5 +226,6 @@
 		<origin xyz="+0.00000000 -0.11400000 +0.08300000" rpy="${PI/2} ${PI/2} 0"/>
 		<axis xyz="0 0 1"/>
-		<limit effort="10" velocity="1" lower="-${175*PI/180}" upper="${175*PI/180}"/>
+		<limit effort="100" velocity="3" lower="-${175*PI/180}" upper="${175*PI/180}"/>
+		<dynamics damping="0.0" friction="0.0"/>
 	</joint>
 	<joint name="joint5" type="revolute">
@@ -229,5 +234,6 @@
 		<origin xyz="-0.16800000 +0.00000000 +0.06900000" rpy="-${PI/2} 0 ${PI/2}"/>
 		<axis xyz="0 0 1"/>
-		<limit effort="10" velocity="1" lower="-${215*PI/180}" upper="${215*PI/180}"/>
+		<limit effort="100" velocity="3" lower="-${215*PI/180}" upper="${215*PI/180}"/>
+		<dynamics damping="0.0" friction="0.0"/>
 	</joint>
 	<joint name="tcp" type="fixed">
@@ -236,63 +242,65 @@
 		<origin xyz="0 0 0.06" rpy="0 0 0"/>
 	</joint>
-	<transmission name="tran0">
-		<type>transmission_interface/SimpleTransmission</type>
-		<joint name="joint0">
-			<hardwareInterface>hardware_interface/PositionJointInterface</hardwareInterface>
-		</joint>
-		<actuator name="motor0">
-			<hardwareInterface>hardware_interface/PositionJointInterface</hardwareInterface>
-			<mechanicalReduction>1</mechanicalReduction>
-		</actuator>
-	</transmission>
-	<transmission name="tran1">
-		<type>transmission_interface/SimpleTransmission</type>
-		<joint name="joint1">
-			<hardwareInterface>hardware_interface/PositionJointInterface</hardwareInterface>
-		</joint>
-		<actuator name="motor1">
-			<hardwareInterface>hardware_interface/PositionJointInterface</hardwareInterface>
-			<mechanicalReduction>1</mechanicalReduction>
-		</actuator>
-	</transmission>
-	<transmission name="tran2">
-		<type>transmission_interface/SimpleTransmission</type>
-		<joint name="joint2">
-			<hardwareInterface>hardware_interface/PositionJointInterface</hardwareInterface>
-		</joint>
-		<actuator name="motor2">
-			<hardwareInterface>hardware_interface/PositionJointInterface</hardwareInterface>
-			<mechanicalReduction>1</mechanicalReduction>
-		</actuator>
-	</transmission>
-	<transmission name="tran3">
-		<type>transmission_interface/SimpleTransmission</type>
-		<joint name="joint3">
-			<hardwareInterface>hardware_interface/PositionJointInterface</hardwareInterface>
-		</joint>
-		<actuator name="motor3">
-			<hardwareInterface>hardware_interface/PositionJointInterface</hardwareInterface>
-			<mechanicalReduction>1</mechanicalReduction>
-		</actuator>
-	</transmission>
-	<transmission name="tran4">
-		<type>transmission_interface/SimpleTransmission</type>
-		<joint name="joint4">
-			<hardwareInterface>hardware_interface/PositionJointInterface</hardwareInterface>
-		</joint>
-		<actuator name="motor4">
-			<hardwareInterface>hardware_interface/PositionJointInterface</hardwareInterface>
-			<mechanicalReduction>1</mechanicalReduction>
-		</actuator>
-	</transmission>
-	<transmission name="tran5">
-		<type>transmission_interface/SimpleTransmission</type>
-		<joint name="joint5">
-			<hardwareInterface>hardware_interface/PositionJointInterface</hardwareInterface>
-		</joint>
-		<actuator name="motor5">
-			<hardwareInterface>hardware_interface/PositionJointInterface</hardwareInterface>
-			<mechanicalReduction>1</mechanicalReduction>
-		</actuator>
-	</transmission>
+	<xacro:macro name="indy7_transmission" params="hw_interface">
+		<transmission name="tran0">
+			<type>transmission_interface/SimpleTransmission</type>
+			<joint name="joint0">
+				<hardwareInterface>${hw_interface}</hardwareInterface>
+			</joint>
+			<actuator name="motor0">
+				<hardwareInterface>${hw_interface}</hardwareInterface>
+				<mechanicalReduction>1</mechanicalReduction>
+			</actuator>
+		</transmission>
+		<transmission name="tran1">
+			<type>transmission_interface/SimpleTransmission</type>
+			<joint name="joint1">
+				<hardwareInterface>${hw_interface}</hardwareInterface>
+			</joint>
+			<actuator name="motor1">
+				<hardwareInterface>${hw_interface}</hardwareInterface>
+				<mechanicalReduction>1</mechanicalReduction>
+			</actuator>
+		</transmission>
+		<transmission name="tran2">
+			<type>transmission_interface/SimpleTransmission</type>
+			<joint name="joint2">
+				<hardwareInterface>${hw_interface}</hardwareInterface>
+			</joint>
+			<actuator name="motor2">
+				<hardwareInterface>${hw_interface}</hardwareInterface>
+				<mechanicalReduction>1</mechanicalReduction>
+			</actuator>
+		</transmission>
+		<transmission name="tran3">
+			<type>transmission_interface/SimpleTransmission</type>
+			<joint name="joint3">
+				<hardwareInterface>${hw_interface}</hardwareInterface>
+			</joint>
+			<actuator name="motor3">
+				<hardwareInterface>${hw_interface}</hardwareInterface>
+				<mechanicalReduction>1</mechanicalReduction>
+			</actuator>
+		</transmission>
+		<transmission name="tran4">
+			<type>transmission_interface/SimpleTransmission</type>
+			<joint name="joint4">
+				<hardwareInterface>${hw_interface}</hardwareInterface>
+			</joint>
+			<actuator name="motor4">
+				<hardwareInterface>${hw_interface}</hardwareInterface>
+				<mechanicalReduction>1</mechanicalReduction>
+			</actuator>
+		</transmission>
+		<transmission name="tran5">
+			<type>transmission_interface/SimpleTransmission</type>
+			<joint name="joint5">
+				<hardwareInterface>${hw_interface}</hardwareInterface>
+			</joint>
+			<actuator name="motor5">
+				<hardwareInterface>${hw_interface}</hardwareInterface>
+				<mechanicalReduction>1</mechanicalReduction>
+			</actuator>
+		</transmission>
+	</xacro:macro>
 </robot>

File: docker/docker_containers/indy7_container/share/catkin_ws/src/indy-ros/indy7_description/urdf/indy7_fixed.xacro (robot description, xacro)
@@ -2,4 +2,5 @@
 <robot name="indy7" xmlns:xacro="http://ros.org/wiki/xacro">
   	<xacro:include filename="$(find indy7_description)/urdf/indy7.xacro"/>
+	<xacro:indy7_transmission hw_interface="hardware_interface/VelocityJointInterface" />
 	<link name="world"/>
     <joint name="global" type="fixed">
