Commit message: unity teleoperation

File: docker/docker_containers/indy7_container/share/catkin_ws/src/indy-ros/indy7_description/urdf/indy7_fixed.xacro (robot description, xacro)
@@ -7,5 +7,5 @@
 		<parent link="world"/>
 		<child link="link0"/>
-		<origin xyz="0 0 0.1" rpy="0 0 0"/>
+		<origin xyz="0 0 0.1" rpy="0 0 -1.57"/>
 	</joint>
 </robot>
